Commit message: add sailboat_gazebo_plugins

File: Gazebo/sailboat_gazebo/urdf/imu.xacro (robot description, xacro)
@@ -27,4 +27,5 @@
       <alwaysOn>true</alwaysOn>
       <bodyName>base_link</bodyName>
+      <frameName>base_link</frameName>
       <topicName>imu</topicName>
       <serviceName>imu_service</serviceName>

File: Gazebo/sailboat_gazebo/urdf/sailboat_base.xacro (robot description, xacro)
@@ -36,5 +36,5 @@
   <link name="base_link">
     <inertial>
-      <mass value="29" />
+      <mass value="15.3" />
       <!--This is the pose of the inertial reference frame, relative to the link reference frame. The origin of the inertial reference frame needs to be at the center of gravity. The axes of the inertial reference frame do not need to be aligned with the principal axes of the inertia.-->
       <origin xyz="0 0 0" />

File: Gazebo/sailboat_gazebo/urdf/sailboat_gazebo.xacro (robot description, xacro)
@@ -6,4 +6,5 @@
     <!-- Defines the "usv_gazebo" macro which implements the plugin for USV dynamics -->
     <xacro:include filename="$(find usv_gazebo_plugins)/urdf/usv_gazebo_dynamics_plugin.xacro" />
+    <xacro:include filename="$(find sailboat_gazebo_plugins)/urdf/sailboat_gazebo_dynamics_plugin.xacro" />
     <!-- Defines the macro for simulated GPS -->
     <xacro:include filename="$(find sailboat_gazebo)/urdf/gps.xacro" />
@@ -18,5 +19,5 @@
     <xacro:sailboat_base />
     <!-- USV dynamic model -->
-    <xacro:usv_gazebo name="sailboat"/>
+    <xacro:sailboat_gazebo name="sailboat"/>
     <!-- Optional sensor plugins - called by macros defined above -->
     <xacro:sailboat_gps_gazebo name="sailboat"/>
