Commit message: modify usv gazebo

File: Gazebo/sailboat_gazebo/urdf/materials.xacro (robot description, xacro)
@@ -1,28 +1,3 @@
 <?xml version="1.0"?>
-<!--
-Copyright (c) 2013 Clearpath Robotics
-All rights reserved.
-Redistribution and use in source and binary forms, with or without
-modification, are permitted provided that the following conditions are met:
-    * Redistributions of source code must retain the above copyright
-      notice, this list of conditions and the following disclaimer.
-    * Redistributions in binary form must reproduce the above copyright
-      notice, this list of conditions and the following disclaimer in the
-      documentation and/or other materials provided with the distribution.
-    * Neither the name of Clearpath Robotics nor the
-      names of its contributors may be used to endorse or promote products
-      derived from this software without specific prior written permission.
-THIS SOFTWARE IS PROVIDED BY THE COPYRIGHT HOLDERS AND CONTRIBUTORS "AS IS" AND
-ANY EXPRESS OR IMPLIED WARRANTIES, INCLUDING, BUT NOT LIMITED TO, THE IMPLIED
-WARRANTIES OF MERCHANTABILITY AND FITNESS FOR A PARTICULAR PURPOSE ARE
-DISCLAIMED. IN NO EVENT SHALL THE COPYRIGHT HOLDERS BE LIABLE FOR ANY
-DIRECT, INDIRECT, INCIDENTAL, SPECIAL, EXEMPLARY, OR CONSEQUENTIAL DAMAGES
-(INCLUDING, BUT NOT LIMITED TO, PROCUREMENT OF SUBSTITUTE GOODS OR SERVICES;
-LOSS OF USE, DATA, OR PROFITS; OR BUSINESS INTERRUPTION) HOWEVER CAUSED AND
-ON ANY THEORY OF LIABILITY, WHETHER IN CONTRACT, STRICT LIABILITY, OR TORT
-(INCLUDING NEGLIGENCE OR OTHERWISE) ARISING IN ANY WAY OUT OF THE USE OF THIS
-SOFTWARE, EVEN IF ADVISED OF THE POSSIBILITY OF SUCH DAMAGE.
-This program contains the materials for the Clearpath Kingfisher model.
--->
 <robot>
 	<material name="Black">

File: Gazebo/usv_gazebo/urdf/base_gazebo.xacro (robot description, xacro)
@@ -1,14 +1,14 @@
 <?xml version="1.0"?>
 <robot xmlns:xacro="http://ros.org/wiki/xacro"
-       name="kingfisher">
-  <!-- Defines the "kingfisher_base" macro -->
-  <xacro:include filename="$(find usv_gazebo)/urdf/kingfisher_urdf.xacro" />
-  <!--<xacro:include filename="$(find usv_gazebo)/urdf/kingfisher_urdf_camera.xacro" />-->
+       name="usv">
+  <!-- Defines the "usv_base" macro -->
+  <xacro:include filename="$(find usv_gazebo)/urdf/usv_urdf.xacro" />
+  <!--<xacro:include filename="$(find usv_gazebo)/urdf/usv_urdf_camera.xacro" />-->
   <!-- Defines the "usv_gazebo" macro which implements the plugin for USV dynamics -->
   <xacro:include filename="$(find usv_gazebo_plugins)/urdf/usv_gazebo_dynamics_plugin.xacro" />
   <!-- Testing old plugin -->
-  <!--<xacro:include filename="$(find kingfisher_plugins)/urdf/kingfisher_plugin.xacro" />-->
+  <!--<xacro:include filename="$(find usv_plugins)/urdf/usv_plugin.xacro" />-->
   <!-- Defines the macro for including simulated camera -->
-  <xacro:include filename="$(find usv_gazebo)/urdf/kingfisher_camera.xacro" />
+  <xacro:include filename="$(find usv_gazebo)/urdf/usv_camera.xacro" />
   <!-- Defines the macro for simulated GPS -->
   <xacro:include filename="$(find usv_gazebo)/urdf/gps_gazebo.xacro" />
@@ -19,17 +19,17 @@
   <!-- Call the macros defined above -->
   <!-- includes basic description witout plugins -->
-  <xacro:kingfisher_base />
+  <xacro:usv_base />
   <!-- USV dynamic model -->
-  <xacro:usv_gazebo name="kingfisher"/>
+  <xacro:usv_gazebo name="usv"/>
   <!-- Optional sensor plugins - called by macros defined above -->
   <xacro:if value="$(arg gps)">
-    <xacro:kingfisher_gps_gazebo name="kingfisher"/>
+    <xacro:usv_gps_gazebo name="usv"/>
   </xacro:if>
   <xacro:if value="$(arg imu)">
-    <xacro:kingfisher_imu_gazebo name="kingfisher"/>
+    <xacro:usv_imu_gazebo name="usv"/>
   </xacro:if>
   <xacro:if value="$(arg p3d)">
-    <xacro:kingfisher_p3d_gazebo name="kingfisher"/>
+    <xacro:usv_p3d_gazebo name="usv"/>
   </xacro:if>
-  <xacro:usv_gazebo_camera name="kingfisher"/>
+  <xacro:usv_gazebo_camera name="usv"/>
 </robot>

File: Gazebo/usv_gazebo/urdf/gps_gazebo.xacro (robot description, xacro)
@@ -1,5 +1,5 @@
 <?xml version="1.0"?>
 <robot xmlns:xacro="http://ros.org/wiki/xacro">
-  <xacro:macro name="kingfisher_gps_gazebo" params="name">
+  <xacro:macro name="usv_gps_gazebo" params="name">
     <gazebo>
       <plugin name="gps_plugin_${name}" filename="libhector_gazebo_ros_gps.so">

File: Gazebo/usv_gazebo/urdf/imu_gazebo.xacro (robot description, xacro)
@@ -1,5 +1,5 @@
 <?xml version="1.0"?>
 <robot xmlns:xacro="http://ros.org/wiki/xacro">
-  <xacro:macro name="kingfisher_imu_gazebo" params="name">
+  <xacro:macro name="usv_imu_gazebo" params="name">
     <gazebo>
       <!-- Either plugin should work -->

File: Gazebo/usv_gazebo/urdf/materials.urdf.xacro (robot description, xacro)
@@ -1,28 +1,3 @@
 <?xml version="1.0"?>
-<!--
-Copyright (c) 2013 Clearpath Robotics
-All rights reserved.
-Redistribution and use in source and binary forms, with or without
-modification, are permitted provided that the following conditions are met:
-    * Redistributions of source code must retain the above copyright
-      notice, this list of conditions and the following disclaimer.
-    * Redistributions in binary form must reproduce the above copyright
-      notice, this list of conditions and the following disclaimer in the
-      documentation and/or other materials provided with the distribution.
-    * Neither the name of Clearpath Robotics nor the
-      names of its contributors may be used to endorse or promote products
-      derived from this software without specific prior written permission.
-THIS SOFTWARE IS PROVIDED BY THE COPYRIGHT HOLDERS AND CONTRIBUTORS "AS IS" AND
-ANY EXPRESS OR IMPLIED WARRANTIES, INCLUDING, BUT NOT LIMITED TO, THE IMPLIED
-WARRANTIES OF MERCHANTABILITY AND FITNESS FOR A PARTICULAR PURPOSE ARE
-DISCLAIMED. IN NO EVENT SHALL THE COPYRIGHT HOLDERS BE LIABLE FOR ANY
-DIRECT, INDIRECT, INCIDENTAL, SPECIAL, EXEMPLARY, OR CONSEQUENTIAL DAMAGES
-(INCLUDING, BUT NOT LIMITED TO, PROCUREMENT OF SUBSTITUTE GOODS OR SERVICES;
-LOSS OF USE, DATA, OR PROFITS; OR BUSINESS INTERRUPTION) HOWEVER CAUSED AND
-ON ANY THEORY OF LIABILITY, WHETHER IN CONTRACT, STRICT LIABILITY, OR TORT
-(INCLUDING NEGLIGENCE OR OTHERWISE) ARISING IN ANY WAY OUT OF THE USE OF THIS
-SOFTWARE, EVEN IF ADVISED OF THE POSSIBILITY OF SUCH DAMAGE.
-This program contains the materials for the Clearpath Kingfisher model.
--->
 <robot>
 	<material name="Black">

File: Gazebo/usv_gazebo/urdf/p3d_gazebo.xacro (robot description, xacro)
@@ -1,5 +1,5 @@
 <?xml version="1.0"?>
 <robot xmlns:xacro="http://ros.org/wiki/xacro">
-  <xacro:macro name="kingfisher_p3d_gazebo" params="name">
+  <xacro:macro name="usv_p3d_gazebo" params="name">
     <gazebo>
       <plugin name="p3d_plugin_${name}" filename="libgazebo_ros_p3d.so">

File: Gazebo/usv_gazebo/urdf/parts.mininertia.urdf.xacro (robot description, xacro)
@@ -1,39 +1,7 @@
 <?xml version="1.0"?>
-<!-- Modified to minimize inertia terms
-Brian Bingham
-Jan, 2017
-Original copyright below-->
-<!--
-Copyright (c) 2012, Ryan Gariepy
-All rights reserved.
-Redistribution and use in source and binary forms, with or without
-modification, are permitted provided that the following conditions are met:
-    * Redistributions of source code must retain the above copyright
-      notice, this list of conditions and the following disclaimer.
-    * Redistributions in binary form must reproduce the above copyright
-      notice, this list of conditions and the following disclaimer in the
-      documentation and/or other materials provided with the distribution.
-    * Neither the name of Clearpath Robotics nor the
-      names of its contributors may be used to endorse or promote products
-      derived from this software without specific prior written permission.
-THIS SOFTWARE IS PROVIDED BY THE COPYRIGHT HOLDERS AND CONTRIBUTORS "AS IS" AND
-ANY EXPRESS OR IMPLIED WARRANTIES, INCLUDING, BUT NOT LIMITED TO, THE IMPLIED
-WARRANTIES OF MERCHANTABILITY AND FITNESS FOR A PARTICULAR PURPOSE ARE
-DISCLAIMED. IN NO EVENT SHALL THE COPYRIGHT HOLDERS BE LIABLE FOR ANY
-DIRECT, INDIRECT, INCIDENTAL, SPECIAL, EXEMPLARY, OR CONSEQUENTIAL DAMAGES
-(INCLUDING, BUT NOT LIMITED TO, PROCUREMENT OF SUBSTITUTE GOODS OR SERVICES;
-LOSS OF USE, DATA, OR PROFITS; OR BUSINESS INTERRUPTION) HOWEVER CAUSED AND
-ON ANY THEORY OF LIABILITY, WHETHER IN CONTRACT, STRICT LIABILITY, OR TORT
-(INCLUDING NEGLIGENCE OR OTHERWISE) ARISING IN ANY WAY OUT OF THE USE OF THIS
-SOFTWARE, EVEN IF ADVISED OF THE POSSIBILITY OF SUCH DAMAGE.
-This program is a macro for adding decorative parts to the Clearpath Kingfisher M200 model.
-It is assumed that such parts are fixed to others, and those other parts' inertial
-parameters account for the decorative parts. Decorative parts currently do not
-incorporate collision.
--->
 <robot xmlns:sensor="http://playerstage.sourceforge.net/gazebo/xmlschema/#sensor"
 	xmlns:controller="http://playerstage.sourceforge.net/gazebo/xmlschema/#controller"
 	xmlns:interface="http://playerstage.sourceforge.net/gazebo/xmlschema/#interface"
-	xmlns:xacro="http://ros.org/wiki/xacro" name="kingfisher_part">
+	xmlns:xacro="http://ros.org/wiki/xacro" name="usv_part">
 	<xacro:property name="x_com" value="0.00000000" /> <!-- com : center of mass -->
 	<xacro:property name="y_com" value="0.00000000" /> <!-- com : center of mass -->
@@ -50,5 +18,5 @@
 	<xacro:property name="iyz_com_cs" value="0.00" /> <!-- at center of mass aligned with coordinate system, kg*m^2-->
 	<xacro:property name="izz_com_cs" value="${min_inertia}" /> <!-- at center of mass aligned with coordinate system, kg*m^2-->
-	<xacro:macro name="kingfisher_part" params="parent name mesh translateX translateY translateZ rotateX rotateY rotateZ color">
+	<xacro:macro name="usv_part" params="parent name mesh translateX translateY translateZ rotateX rotateY rotateZ color">
 		<joint name="${parent}_${name}_joint" type="fixed">
 		    <origin xyz="${translateX} ${translateY} ${translateZ}"

File: Gazebo/usv_gazebo/urdf/parts.urdf.xacro (robot description, xacro)
@@ -1,35 +1,7 @@
 <?xml version="1.0"?>
-<!--
-Copyright (c) 2012, Ryan Gariepy
-All rights reserved.
-Redistribution and use in source and binary forms, with or without
-modification, are permitted provided that the following conditions are met:
-    * Redistributions of source code must retain the above copyright
-      notice, this list of conditions and the following disclaimer.
-    * Redistributions in binary form must reproduce the above copyright
-      notice, this list of conditions and the following disclaimer in the
-      documentation and/or other materials provided with the distribution.
-    * Neither the name of Clearpath Robotics nor the
-      names of its contributors may be used to endorse or promote products
-      derived from this software without specific prior written permission.
-THIS SOFTWARE IS PROVIDED BY THE COPYRIGHT HOLDERS AND CONTRIBUTORS "AS IS" AND
-ANY EXPRESS OR IMPLIED WARRANTIES, INCLUDING, BUT NOT LIMITED TO, THE IMPLIED
-WARRANTIES OF MERCHANTABILITY AND FITNESS FOR A PARTICULAR PURPOSE ARE
-DISCLAIMED. IN NO EVENT SHALL THE COPYRIGHT HOLDERS BE LIABLE FOR ANY
-DIRECT, INDIRECT, INCIDENTAL, SPECIAL, EXEMPLARY, OR CONSEQUENTIAL DAMAGES
-(INCLUDING, BUT NOT LIMITED TO, PROCUREMENT OF SUBSTITUTE GOODS OR SERVICES;
-LOSS OF USE, DATA, OR PROFITS; OR BUSINESS INTERRUPTION) HOWEVER CAUSED AND
-ON ANY THEORY OF LIABILITY, WHETHER IN CONTRACT, STRICT LIABILITY, OR TORT
-(INCLUDING NEGLIGENCE OR OTHERWISE) ARISING IN ANY WAY OUT OF THE USE OF THIS
-SOFTWARE, EVEN IF ADVISED OF THE POSSIBILITY OF SUCH DAMAGE.
-This program is a macro for adding decorative parts to the Clearpath Kingfisher M200 model.
-It is assumed that such parts are fixed to others, and those other parts' inertial
-parameters account for the decorative parts. Decorative parts currently do not
-incorporate collision.
--->
 <robot xmlns:sensor="http://playerstage.sourceforge.net/gazebo/xmlschema/#sensor"
 	xmlns:controller="http://playerstage.sourceforge.net/gazebo/xmlschema/#controller"
 	xmlns:interface="http://playerstage.sourceforge.net/gazebo/xmlschema/#interface"
-	xmlns:xacro="http://ros.org/wiki/xacro" name="kingfisher_part">
+	xmlns:xacro="http://ros.org/wiki/xacro" name="usv_part">
 	<property name="x_com" value="0.00000000" /> <!-- com : center of mass -->
 	<property name="y_com" value="0.00000000" /> <!-- com : center of mass -->
@@ -45,5 +17,5 @@
 	<property name="iyz_com_cs" value="0.00" /> <!-- at center of mass aligned with coordinate system, kg*m^2-->
 	<property name="izz_com_cs" value="0.01" /> <!-- at center of mass aligned with coordinate system, kg*m^2-->
-	<xacro:macro name="kingfisher_part" params="parent name mesh translateX translateY translateZ rotateX rotateY rotateZ color">
+	<xacro:macro name="usv_part" params="parent name mesh translateX translateY translateZ rotateX rotateY rotateZ color">
 		<joint name="${parent}_${name}_joint" type="fixed">
 		    <origin xyz="${translateX} ${translateY} ${translateZ}"

File: Gazebo/usv_gazebo/urdf/usv_gazebo.xacro (robot description, xacro)
@@ -2,5 +2,5 @@
 <robot xmlns:xacro="http://ros.org/wiki/xacro">
   <xacro:macro name="usv_gazebo" params="name">
-    <!--Gazebo Plugin for simulating Kingfisher dynamics-->
+    <!--Gazebo Plugin for simulating usv dynamics-->
     <gazebo>
       <!--<plugin name="heron_dynamic" filename="libheron_gazebo_plugins.so">-->

File: Gazebo/usv_gazebo/urdf/usv_urdf.xacro (robot description, xacro)
@@ -1,37 +1,8 @@
 <?xml version="1.0"?>
-<!-- Modified to minimize inertia terms
-Brian Bingham
-Jan, 2017
-Original copyright below-->
-<!--
-Copyright (c) 2012, Clearpath Robotics
-All rights reserved.
-Redistribution and use in source and binary forms, with or without
-modification, are permitted provided that the following conditions are met:
-    * Redistributions of source code must retain the above copyright
-      notice, this list of conditions and the following disclaimer.
-    * Redistributions in binary form must reproduce the above copyright
-      notice, this list of conditions and the following disclaimer in the
-      documentation and/or other materials provided with the distribution.
-    * Neither the name of Clearpath Robotics nor the
-      names of its contributors may be used to endorse or promote products
-      derived from this software without specific prior written permission.
-THIS SOFTWARE IS PROVIDED BY THE COPYRIGHT HOLDERS AND CONTRIBUTORS "AS IS" AND
-ANY EXPRESS OR IMPLIED WARRANTIES, INCLUDING, BUT NOT LIMITED TO, THE IMPLIED
-WARRANTIES OF MERCHANTABILITY AND FITNESS FOR A PARTICULAR PURPOSE ARE
-DISCLAIMED. IN NO EVENT SHALL THE COPYRIGHT HOLDERS BE LIABLE FOR ANY
-DIRECT, INDIRECT, INCIDENTAL, SPECIAL, EXEMPLARY, OR CONSEQUENTIAL DAMAGES
-(INCLUDING, BUT NOT LIMITED TO, PROCUREMENT OF SUBSTITUTE GOODS OR SERVICES;
-LOSS OF USE, DATA, OR PROFITS; OR BUSINESS INTERRUPTION) HOWEVER CAUSED AND
-ON ANY THEORY OF LIABILITY, WHETHER IN CONTRACT, STRICT LIABILITY, OR TORT
-(INCLUDING NEGLIGENCE OR OTHERWISE) ARISING IN ANY WAY OUT OF THE USE OF THIS
-SOFTWARE, EVEN IF ADVISED OF THE POSSIBILITY OF SUCH DAMAGE.
-This program contains the description of the robot base model for the Clearpath Kingfisher
--->
-<robot name="kingfisher" xmlns:xacro="http://ros.org/wiki/xacro">
-  <xacro:macro name="kingfisher_base">
+<robot name="usv" xmlns:xacro="http://ros.org/wiki/xacro">
+  <xacro:macro name="usv_base">
   <!-- Included URDF/XACRO Files -->
   <xacro:include filename="$(find usv_gazebo)/urdf/materials.urdf.xacro" />
-  <!-- Replace original Kingfisher file with new one with minimial inertia-->
+  <!-- Replace original usv file with new one with minimial inertia-->
   <xacro:include filename="$(find usv_gazebo)/urdf/parts.mininertia.urdf.xacro" />
   <!-- PROPERTY LIST -->
@@ -72,5 +43,5 @@
       <origin xyz="0 0 ${HH}" rpy="${M_PI/2} 0 ${M_PI/2}" />
       <geometry>
-	<mesh filename="package://usv_gazebo/meshes/kingfisher_base.stl" />
+	<mesh filename="package://usv_gazebo/meshes/usv_base.stl" />
       </geometry>
       <material name="DarkGray" />
@@ -94,5 +65,5 @@
   <!-- PANEL-LINKS -->
   <!-- Top Plate -->
-  <kingfisher_part parent="base_footprint" name="left_panel" mesh="left_panel"
+  <usv_part parent="base_footprint" name="left_panel" mesh="left_panel"
 		   translateX="0.0" translateY="-0.35" translateZ="${0.05+HH*2}"
 		   rotateX="${M_PI/2}" rotateY="0.0" rotateZ="${M_PI/2}"
@@ -101,5 +72,5 @@
     <material>Gazebo/Yellow</material>
   </gazebo>
-  <kingfisher_part parent="base_footprint" name="right_panel" mesh="right_panel"
+  <usv_part parent="base_footprint" name="right_panel" mesh="right_panel"
 		   translateX="0.0" translateY="0.35" translateZ="${0.05+HH*2}"
 		   rotateX="${M_PI/2}" rotateY="0.0" rotateZ="${-M_PI/2}"

File: Gazebo/usv_gazebo_plugins/urdf/usv_gazebo_dynamics_plugin.xacro (robot description, xacro)
@@ -2,5 +2,5 @@
 <robot xmlns:xacro="http://www.ros.org/wiki/xacro">
   <xacro:macro name="usv_gazebo" params="name">
-    <!--Gazebo Plugin for simulating Kingfisher dynamics-->
+    <!--Gazebo Plugin for simulating usv dynamics-->
     <gazebo >
       <!--<plugin name="heron_dynamic" filename="libheron_gazebo_plugins.so">-->
