Commit message: add gazebo laser plugin

File: Gazebo/sailboat_gazebo/urdf/sailboat_gazebo_laser.xacro (robot description, xacro)
@@ -14,5 +14,5 @@
     <xacro:include filename="$(find sailboat_gazebo)/urdf/camera.xacro" />
     <!-- Defines the macro for simulated laser -->
-    <xacro:include filename="$(find sailboat_gazebo)/urdf/laser.xacro" />
+    <!-- <xacro:include filename="$(find sailboat_gazebo)/urdf/laser.xacro" /> -->
     <!-- Call the macros defined above -->
     <!-- includes basic description witout plugins -->
@@ -24,4 +24,12 @@
     <xacro:sailboat_imu_gazebo name="sailboat"/>
     <xacro:sailboat_camera_gazebo name="sailboat"/>
-    <xacro:sailboat_laser_gazebo name="sailboat"/>
+    <!-- <xacro:sailboat_laser_gazebo name="sailboat"/> -->
+    <!-- <xacro:include filename="$(find velodyne_description)/urdf/VLP-16.urdf.xacro"/>
+    <VLP-16 parent="base_link" name="velodyne" topic="/velodyne_points" hz="10" samples="440">
+       <origin xyz="0 0 0.4" rpy="0 0 0" />
+    </VLP-16> -->
+    <xacro:include filename="$(find velodyne_description)/urdf/HDL-32E.urdf.xacro"/>
+    <HDL-32E parent="base_link" name="velodyne" topic="/velodyne_points2" hz="10" samples="220">
+        <origin xyz="0 0 0.6" rpy="0 0 0" />
+    </HDL-32E>
 </robot>
