Commit message: modify sailboat gazebo

File: Gazebo/sailboat_gazebo/urdf/sailboat_base.xacro (robot description, xacro)
@@ -40,5 +40,6 @@
       <origin xyz="0 0 0" />
       <!--The 3x3 rotational inertia matrix. Because the rotational inertia matrix is symmetric, only 6 above-diagonal elements of this matrix are specified here, using the attributes ixx, ixy, ixz, iyy, iyz, izz.-->
-      <inertia ixx="10" ixy="0" ixz="0" iyy="10" iyz="0" izz="10" />
+      <inertia ixx="5" ixy="0" ixz="0" iyy="10" iyz="0" izz="5" />
+      <!-- <inertia ixx="2.002" ixy="0" ixz="-0.226" iyy="10" iyz="0" izz="1.535" /> -->
     </inertial>
     <visual>
@@ -90,4 +91,25 @@
     <turnGravityOff>false</turnGravityOff>
   </gazebo>
+  <link name="GPS">
+    <visual>
+      <geometry>
+        <cylinder length="0.1" radius="0.05"/>
+      </geometry>
+    </visual>
+  </link>
+  <link name="AHRS">
+    <visual>
+      <geometry>
+        <cylinder length="0.1" radius="0.05"/>
+      </geometry>
+    </visual>
+  </link>
+  <link name="WTST">
+    <visual>
+      <geometry>
+        <cylinder length="0.1" radius="0.05"/>
+      </geometry>
+    </visual>
+  </link>
   <joint name="boat_to_sail" type="fixed">
     <parent link="base_link"/>
@@ -101,4 +123,19 @@
     <axis xyz="0 0 1"/>
     <origin xyz="-0.75 0 -0.1"/>
+  </joint>
+  <joint name="boat_to_GPS" type="fixed">
+    <parent link="base_link"/>
+    <child link="GPS"/>
+    <origin xyz="-0.75 0 0.2"/>
+  </joint>
+  <joint name="boat_to_AHRS" type="fixed">
+    <parent link="base_link"/>
+    <child link="AHRS"/>
+    <origin xyz="0 0 0.2"/>
+  </joint>
+    <joint name="boat_to_WTST" type="fixed">
+    <parent link="base_link"/>
+    <child link="WTST"/>
+    <origin xyz="0.75 0 0.2"/>
   </joint>
   <!-- Define a location for the camera to sit -->

Commit message: test avoidance simulation

File: Gazebo/sailboat_gazebo/urdf/sailboat_base.xacro (robot description, xacro)
@@ -94,5 +94,5 @@
     <visual>
       <geometry>
-        <cylinder length="0.1" radius="0.05"/>
+        <cylinder length="0.01" radius="0.01"/>
       </geometry>
     </visual>
@@ -101,5 +101,5 @@
     <visual>
       <geometry>
-        <cylinder length="0.1" radius="0.05"/>
+        <cylinder length="0.01" radius="0.01"/>
       </geometry>
     </visual>
@@ -108,5 +108,5 @@
     <visual>
       <geometry>
-        <cylinder length="0.1" radius="0.05"/>
+        <cylinder length="0.01" radius="0.01"/>
       </geometry>
     </visual>
@@ -127,5 +127,5 @@
     <parent link="base_link"/>
     <child link="GPS"/>
-    <origin xyz="-0.75 0 0.2"/>
+    <origin xyz="0.5 0 0.2"/>
   </joint>
   <joint name="boat_to_AHRS" type="fixed">
@@ -137,5 +137,5 @@
     <parent link="base_link"/>
     <child link="WTST"/>
-    <origin xyz="0.75 0 0.2"/>
+    <origin xyz="-0.75 0 0.2"/>
   </joint>
   <!-- Define a location for the camera to sit -->
@@ -143,5 +143,5 @@
   <joint name="camera_joint" type="fixed">
     <axis xyz="0 1 0" />
-    <origin xyz="0.32 0 0.2" rpy="0 0 0"/>
+    <origin xyz="0.75 0 0.2" rpy="0 0 0"/>
     <parent link="base_link"/>
     <child link="camera_link"/>
