Commit message: modify usv_gazebo control and urdf

File: Gazebo/usv_gazebo/urdf/gps_gazebo.xacro (robot description, xacro)
@@ -4,19 +4,20 @@
     <gazebo>
       <plugin name="gps_plugin_${name}" filename="libhector_gazebo_ros_gps.so">
-	<updateRate>1.0</updateRate>
-	<alwaysOn>true</alwaysOn>
-	<bodyName>base_link</bodyName>
-	<frameId>base_link</frameId>
-	<topicName>gps/fix</topicName>
-	<velocityTopicName>fix_velocity</velocityTopicName>
-	<referenceLatitude>36.6</referenceLatitude>
-	<referenceLongitude>-121.9</referenceLongitude>
-	<referenceAltitude>10.0</referenceAltitude>
-	<offset>0.0 0.0 0.0</offset>
-	<drift>0.0 0.0 0.0</drift>
-	<gaussianNoise>0.1 0.1 0.1</gaussianNoise>
-	<velocityOffset>0.0 0.0 0.0</velocityOffset>
-	<velocityDrift>0.0 0.0 0.0</velocityDrift>
-	<velocityGaussianNoise>0.0 0.0 0.0</velocityGaussianNoise>
+          <updateRate>1.0</updateRate>
+		      <alwaysOn>true</alwaysOn>
+          <bodyName>base_link</bodyName>
+          <frameId>base_link</frameId>
+          <topicName>/gps/fix</topicName>
+          <velocityTopicName>/gps/fix_velocity</velocityTopicName>
+          <referenceLatitude>-30.06022459407145675</referenceLatitude>
+          <referenceLongitude>-51.173913575780311191</referenceLongitude>
+          <referenceHeading>90</referenceHeading>
+          <referenceAltitude>10</referenceAltitude>
+          <offset>0 0 0</offset>
+          <drift>0.001 0.001 0.001</drift>
+          <gaussianNoise>0.05 0.05 0.05</gaussianNoise>
+		      <velocityOffset>0.0 0.0 0.0</velocityOffset>
+          <velocityDrift>0 0 0</velocityDrift>
+          <velocityGaussianNoise>0.05 0.05 0.05</velocityGaussianNoise>
       </plugin>
     </gazebo>

File: Gazebo/usv_gazebo/urdf/imu_gazebo.xacro (robot description, xacro)
@@ -5,24 +5,13 @@
       <!-- Either plugin should work -->
       <!--<plugin name="imu_plugin_${name}" filename="libgazebo_ros_imu.so">-->
-      <plugin name="imu_plugin_${name}" filename="libhector_gazebo_ros_imu.so">
-	<updateRate>10.0</updateRate>
-	<bodyName>base_link</bodyName>
-	<topicName>imu/data</topicName>
-	<serviceName>imu_service</serviceName>
-	<frame_id>odom</frame_id>
-	<alwaysOn>true</alwaysOn>
-	<accelOffset>0.0 0.0 0.0</accelOffset>
-	<accelDrift>0.0 0.0 0.0</accelDrift>
-	<accelDriftFrequency>0.00027 0.00027 0.000027</accelDriftFrequency>
-	<accelGaussianNoise>0.0 0.0 0.0</accelGaussianNoise>
-	<rateOffset>0.0 0.0 0.0</rateOffset>
-	<rateDrift>0.0 0.0 0.0</rateDrift>
-	<rateDriftFrequency>0.00027 0.00027 0.000027</rateDriftFrequency>
-	<rateGaussianNoise>0.0 0.0 0.0</rateGaussianNoise>
-	<yawOffset>0.0</yawOffset>
-	<yawDrift>0.0</yawDrift>
-	<yawDriftFrequency>0.00027</yawDriftFrequency>
-	<yawGaussianNoise>0.0</yawGaussianNoise>
-      </plugin>
+    <plugin name="imu_plugin_${name}" filename="libgazebo_ros_imu.so">
+      <alwaysOn>true</alwaysOn>
+      <bodyName>base_link</bodyName>
+      <frameName>base_link</frameName>
+      <topicName>imu</topicName>
+      <serviceName>imu_service</serviceName>
+      <gaussianNoise>0.0</gaussianNoise>
+      <updateRate>20.0</updateRate>
+    </plugin>
     </gazebo>
   </xacro:macro>

File: Gazebo/usv_gazebo/urdf/usv_gazebo_laser.xacro (robot description, xacro)
@@ -10,5 +10,5 @@
   <!--<xacro:include filename="$(find usv_plugins)/urdf/usv_plugin.xacro" />-->
   <!-- Defines the macro for including simulated camera -->
-  <xacro:include filename="$(find usv_gazebo)/urdf/usv_camera.xacro" />
+  <xacro:include filename="$(find usv_gazebo)/urdf/camera_gazebo.xacro" />
   <!-- Defines the macro for simulated GPS -->
   <xacro:include filename="$(find usv_gazebo)/urdf/gps_gazebo.xacro" />
@@ -16,5 +16,5 @@
   <xacro:include filename="$(find usv_gazebo)/urdf/imu_gazebo.xacro" />
   <!-- Macro for P3D ground truth -->
-  <xacro:include filename="$(find usv_gazebo)/urdf/p3d_gazebo.xacro" />
+  <!-- <xacro:include filename="$(find usv_gazebo)/urdf/p3d_gazebo.xacro" /> -->
   <!-- Call the macros defined above -->
   <!-- includes basic description witout plugins -->
@@ -29,7 +29,11 @@
     <xacro:usv_imu_gazebo name="usv"/>
   </xacro:if>
-  <xacro:if value="$(arg p3d)">
+  <!-- <xacro:if value="$(arg p3d)">
     <xacro:usv_p3d_gazebo name="usv"/>
-  </xacro:if>
+  </xacro:if> -->
   <xacro:usv_gazebo_camera name="usv"/>
+  <xacro:include filename="$(find velodyne_description)/urdf/HDL-32E.urdf.xacro"/>
+  <HDL-32E parent="base_link" name="velodyne" topic="/velodyne_points2" hz="10" samples="220">
+        <origin xyz="0 0 0.6" rpy="0 0 0" />
+  </HDL-32E>
 </robot>
