Commit message: modify detection

File: Gazebo/usv_gazebo/urdf/usv_urdf.xacro (robot description, xacro)
@@ -83,5 +83,5 @@
   <joint name="camera_joint" type="fixed">
     <axis xyz="0 1 0" />
-    <origin xyz="0.32 0 0.2" rpy="0 0 0"/>
+    <origin xyz="0.32 0 0.5" rpy="0 0 0"/>
     <parent link="base_link"/>
     <child link="camera_link"/>
