Commit message: modify sh

File: Common/sailboat_tf_tree/urdf/sailboat001.urdf (robot description, URDF)
Before this commit: robot sailboat001, 6 links, 5 joints
Links:
- added link camera_link; visual box size=0.05 0.05 0.05
- added link laser_link; visual box size=0.05 0.05 0.05
Joints:
- added joint camera_joint: type fixed, parent base_link, child camera_link, origin xyz=0.75 0 0.2 rpy=0 0 0, axis 0 1 0
- added joint laser_joint: type fixed, parent base_link, child laser_link, origin xyz=0.0 0 0.2 rpy=0 0 0, axis 0 1 0
- joint boat_to_GPS: origin xyz=-0.75 0 0.2 -> xyz=0.5 0 0.2
- joint boat_to_WTST: origin xyz=0.75 0 0.2 -> xyz=-0.75 0 0.2
